File: shield-arduino-fashion.kicad_pcb (KiCad board)
At the start: 2 copper layers, 68.6 x 53.3 mm, 14 parts, among them CON1 282834-2, U1 TLE6209R

Commit message: Clean project
Parts:
- removed C1, C3: 100uF/50V, Smd_Electrolytic:100uF_50V_Size_C_8x10
- removed C2: 100n, Capacitors_Smd_0603:100nF_0603
- removed C4: 33nF/50V, Capacitors_Smd_0603:33nF_0603
- removed CON1: 282834-2, TerminalBlock_P2.54:282834-2
- removed D3: FYLS-0805URC, Diodes:FYLS-0805URC
- removed D4: FYLS-0805PGC, Diodes:FYLS-0805PGC
- removed R7, R8: 1k, Resistor_Smd_0603:1k_0603
- removed U1: TLE6209R, H_Bridges_Drivers:TLE6209R
Connections:
- XA1 pad 5V1: 5V -> unconnected-(XA1-Pad5V1)
- XA1 pad VIN: /VIN -> unconnected-(XA1-PadVIN)
Routing:
- net /VIN: track 83.5 -> 0.00 mm
- net 5V: track 64.4 -> 0.00 mm, vias 1 -> 0
- net /SPI_MOSI: track 54.4 -> 0.00 mm, vias 1 -> 0
- net /SPI_SCLK: track 53.1 -> 0.00 mm, vias 1 -> 0
- net /SPI_MISO: track 49.3 -> 0.00 mm, vias 1 -> 0
- net /INH: track 43.8 -> 0.00 mm
- net /SPI_CSN: track 43.2 -> 0.00 mm, vias 1 -> 0
- net /PWM: track 41.7 -> 0.00 mm, vias 2 -> 0
- net /DIS: track 23.3 -> 0.00 mm
- net /DIR: track 22.8 -> 0.00 mm
- net GND: track 12.3 -> 0.00 mm, vias 1 -> 0
- net Net-(CON1-Pad2): track 9.74 -> 0.00 mm
- net Net-(C4-Pad1): track 1.99 -> 0.00 mm
- net Net-(CON1-Pad1): track 1.47 -> 0.00 mm
- net Net-(D4-Pad1): track 1.41 -> 0.00 mm
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- removed copper zone on F.Cu, net Net-(CON1-Pad1)
- removed copper zone on F.Cu, net Net-(CON1-Pad2)
Other:
- board text added: "SOFJAN 2022 ARDUINO SHIELD TEMPLATE"
- board text removed: "OUT1"
- board text removed: "OUT2"
- board text removed: "SOFJAN 2022 FULL BRIDGE TEST BOARD V1.0 NCP5106B"
