File: shield-arduino-fashion.kicad_sch (KiCad schematic)
At the start: 14 parts, among them CON1 282834-2

Commit message: Clean project
Parts:
- removed C1: (no value), Smd_Electrolytic:100uF_50V_Size_C_8x10, symbol Capacitors_Smd_Electrolytic:100uF_50V
- removed C2: (no value), symbol Capacitors_Smd0603:100n
- removed C3: (no value), symbol Capacitors_Smd_Electrolytic:100uF_50V
- removed C4: (no value), symbol Capacitors_Smd0603:33nF
- removed CON1: 282834-2, TerminalBlock_P2.54:282834-2, symbol Terminal_Blocks:282834-2
- removed D3: FYLS-0805URC, Diodes:FYLS-0805URC, symbol Diodes:FYLS-0805URC
- removed D4: FYLS-0805PGC, Diodes:FYLS-0805PGC, symbol Diodes:FYLS-0805PGC
- removed R7, R8: 1k, Resistor_Smd_0603:1k_0603, symbol Resistors_Smd0603:1k
- removed U1: (no value), H_Bridges_Drivers:TLE6209R, symbol H_Bridges_Drivers:TLE6209R
Connections:
- net 5V: no longer names the net of XA1.5V1 (5V)
- net VIN: no longer names the net of XA1.VIN
Other:
- title: Full Bridge based on TLE6209R -> Arduino Shield Template
